Commit message: Add GPS to Simulation
A gps is now simulated in gazebo.

File: src/turtlebot_description/urdf/turtlebot_gazebo.urdf.xacro (robot description, xacro)
@@ -40,3 +40,20 @@
     </gazebo>
   </xacro:macro>
+  <xacro:macro name="turtlebot_robot_position_gazebo">
+    <gazebo>
+      <plugin name="gps_controller" filename="libhector_gazebo_ros_gps.so">
+        <updateRate>40</updateRate>
+        <robotNamespace>/</robotNamespace>
+        <bodyName>base_link</bodyName>
+        <frameId>base_link</frameId>
+        <topicName>navsat/fix</topicName>
+        <velocityTopicName>navsat/vel</velocityTopicName>
+        <referenceLatitude>49.9</referenceLatitude>
+        <referenceLongitude>8.9</referenceLongitude>
+        <referenceHeading>0</referenceHeading>
+        <referenceAltitude>0</referenceAltitude>
+        <drift>0.0001 0.0001 0.0001</drift>
+      </plugin>
+    </gazebo>
+  </xacro:macro>
 </robot>

File: src/turtlebot_description/urdf/turtlebot_library.urdf.xacro (robot description, xacro)
@@ -16,3 +16,5 @@
   <xacro:include filename="$(find turtlebot_description)/urdf/sensors/asus_xtion_pro.urdf.xacro"/>
   <xacro:include filename="$(find turtlebot_description)/urdf/sensors/asus_xtion_pro_offset.urdf.xacro"/>
+  <!-- Additional Sensors for Gazebo -->
+  <turtlebot_robot_position_gazebo/>
 </robot>

Commit message: Add Hokuyo Laser to Gazebo
The lidar is now simulated in gazebo and is in place of the kinect
which in reality would not work outside.  I also added robot state
publisher to get a tf tree generated.

File: src/turtlebot_description/urdf/turtlebot_gazebo.urdf.xacro (robot description, xacro)
@@ -57,3 +57,40 @@
     </gazebo>
   </xacro:macro>
+  <xacro:macro name="turtlebot_sim_laser">
+    <gazebo reference="camera_link">
+    <sensor type="gpu_ray" name="head_hokuyo_sensor">
+      <pose>0 0 0 0 0 0</pose>
+      <visualize>false</visualize>
+      <update_rate>40</update_rate>
+      <ray>
+        <scan>
+          <horizontal>
+            <samples>720</samples>
+            <resolution>1</resolution>
+            <min_angle>-1.570796</min_angle>
+            <max_angle>1.570796</max_angle>
+          </horizontal>
+        </scan>
+        <range>
+          <min>0.3</min>
+          <max>30.0</max>
+          <resolution>0.01</resolution>
+        </range>
+        <noise>
+          <type>gaussian</type>
+          <!-- Noise parameters based on published spec for Hokuyo laser
+               achieving "+-30mm" accuracy at range < 10m.  A mean of 0.0m and
+               stddev of 0.01m will put 99.7% of samples within 0.03m of the true
+               reading. -->
+          <mean>0.0</mean>
+          <stddev>0.01</stddev>
+        </noise>
+      </ray>
+      <plugin name="gazebo_ros_head_hokuyo_controller" filename="libgazebo_ros_gpu_laser.so">
+        <topicName>/laser/scan</topicName>
+        <frameName>camera_link</frameName>
+      </plugin>
+    </sensor>
+  </gazebo>
+  </xacro:macro>
 </robot>

File: src/turtlebot_description/urdf/turtlebot_library.urdf.xacro (robot description, xacro)
@@ -18,3 +18,4 @@
   <!-- Additional Sensors for Gazebo -->
   <turtlebot_robot_position_gazebo/>
+  <turtlebot_sim_laser/>
 </robot>
